Commit message: ll

File: hello_robot_description/urdf/hello_robot.urdf.xacro (robot description, xacro)
@@ -8,6 +8,6 @@
   <xacro:property name="sensor_yaml" value="$(find ${package_name})/config/sensors.yaml" />
   <xacro:property name="sensor_prop" value="${load_yaml(sensor_yaml)}"/>
-  <xacro:property name="baselen" value="0.260" />
-  <xacro:property name="basewidth" value="0.152" />
+  <xacro:property name="baselen" value="0.3" />
+  <xacro:property name="basewidth" value="0.33" />
   <xacro:property name="basethick" value="0.003" />
   <xacro:property name="wheeldiam" value="0.056" />
@@ -28,5 +28,6 @@
     <visual>
       <geometry>
-        <box size="${baselen} ${basewidth} ${basethick}" />
+      <mesh
+          filename="package://hospi_bot/meshes/base_link.STL" />
       </geometry>
       <material name="white"/>
@@ -34,5 +35,6 @@
     <collision>
       <geometry>
-        <box size="${baselen*collision_inflation} ${basewidth*collision_inflation} ${basethick*collision_inflation}" />
+        <mesh
+          filename="package://hospi_bot/meshes/base_link.STL" />
       </geometry>
     </collision>

File: hello_robot_description/urdf/include/common_sensors.xacro (robot description, xacro)
@@ -9,5 +9,6 @@
         <origin xyz="0 0 0" rpy="0 0 0"/>
         <geometry>
-          <mesh filename="package://${package_name}/meshes/sensors/${mesh}" />
+           <mesh
+          filename="package://hospi_bot/meshes/Camera_Link.STL" />
         </geometry>
         <material name="dark_grey"/>
@@ -18,5 +19,6 @@
         <origin xyz="0 0 0" rpy="0 0 0"/>
          <geometry>
-         <cylinder radius="${sensor_prop['gpu_laser']['radius']}" length="${sensor_prop['gpu_laser']['length']}"/>
+          <mesh
+          filename="package://hospi_bot/meshes/Camera_Link.STL" />
         </geometry>
         <material name="red"/>
@@ -26,5 +28,6 @@
         <origin xyz="0 0 0" rpy="0 0 0"/>
         <geometry>
-          <cylinder radius="${sensor_prop['gpu_laser']['radius']}" length="${sensor_prop['gpu_laser']['length']}"/>
+          <mesh
+          filename="package://hospi_bot/meshes/Camera_Link.STL" />
         </geometry>
       </collision>
@@ -42,5 +45,5 @@
     <parent link="${parent_link}"/>
     <child link="${prefix}_gpu_laser_link"/>
-    <origin xyz="${sensor_prop['gpu_laser']['dx']} ${sensor_prop['gpu_laser']['dy']} ${sensor_prop['gpu_laser']['dz']}" rpy="0 0 0"/>
+    <origin xyz="0.17752 -0.00081488 0.235" rpy="0 0 0"/>
     <axis xyz="0 1 0" />
   </joint>
@@ -49,5 +52,5 @@
     <sensor type="ray" name="head_hokuyo_sensor">
       <pose>0 0 0 0 0 0</pose>
-      <visualize>true</visualize>
+      <visualize>false</visualize>
       <update_rate>40</update_rate>
       <ray>
